File: CESP.kicad_pcb (KiCad board)
At the start: 2 copper layers, 55.9 x 44.7 mm, 9 parts

Commit message: ADDED/REMOVED SHIT
Parts:
- removed the LED-1206 at (164.0, 135.9)
- removed the SM0603 at (199.8, 120.8)
Changed lines of the file:
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@@
-(kicad_pcb (version 3) (host pcbnew "(2013-03-19 BZR 4004)-stable")
+(kicad_pcb (version 3) (host pcbnew "(2013-07-07 BZR 4022)-stable")
   (general
     (links 0)
     (no_connects 0)
-    (area 0 0 0 0)
+    (area 154.624316 83.566 213.421684 140.537001)
     (thickness 1.6)
     (drawings 5)
     (tracks 0)
     (zones 0)
-    (modules 9)
+    (modules 7)
     (nets 1)
   )
@@
     (pad_to_mask_clearance 0)
     (aux_axis_origin 0 0)
-    (visible_elements FFFFFFBF)
+    (visible_elements 7FFFFFFF)
     (pcbplotparams
       (layerselection 3178497)
       (usegerberextensions true)
       (excludeedgelayer true)
-      (linewidth 152400)
+      (linewidth 0.150000)
       (plotframeref false)
       (viasonmask false)
@@
   (module SM0603 (layer F.Cu)
     (at 188.214 111.506)
-    (attr smd)
-    (fp_text reference SM0603 (at 0 0) (layer F.SilkS)
-      (effects (font (size 0.508 0.4572) (thickness 0.1143)))
-    )
-    (fp_text value Val** (at 0 0) (layer F.SilkS) hide
-      (effects (font (size 0.508 0.4572) (thickness 0.1143)))
-    )
-    (fp_line (start -1.143 -0.635) (end 1.143 -0.635) (layer F.SilkS) (width 0.127))
-    (fp_line (start 1.143 -0.635) (end 1.143 0.635) (layer F.SilkS) (width 0.127))
-    (fp_line (start 1.143 0.635) (end -1.143 0.635) (layer F.SilkS) (width 0.127))
-    (fp_line (start -1.143 0.635) (end -1.143 -0.635) (layer F.SilkS) (width 0.127))
-    (pad 1 smd rect (at -0.762 0) (size 0.635 1.143)
-      (layers F.Cu F.Paste F.Mask)
-    )
-    (pad 2 smd rect (at 0.762 0) (size 0.635 1.143)
-      (layers F.Cu F.Paste F.Mask)
-    )
-    (model smd\resistors\R0603.wrl
-      (at (xyz 0 0 0.001))
-      (scale (xyz 0.5 0.5 0.5))
-      (rotate (xyz 0 0 0))
-    )
-  )
-  (module SM0603 (layer F.Cu)
-    (at 199.771 120.777)
     (attr smd)
     (fp_text reference SM0603 (at 0 0) (layer F.SilkS)
@@
     (descr "LED 1206 smd package")
     (tags "LED1206 SMD")
-    (attr smd)
-    (fp_text reference LED-1206 (at 0.254 -1.524) (layer F.SilkS)
-      (effects (font (size 0.762 0.762) (thickness 0.0889)))
-    )
-    (fp_text value VAL** (at 0 1.524) (layer F.SilkS)
-      (effects (font (size 0.762 0.762) (thickness 0.0889)))
-    )
-    (fp_line (start -0.09906 0.09906) (end 0.09906 0.09906) (layer F.SilkS) (width 0.06604))
-    (fp_line (start 0.09906 0.09906) (end 0.09906 -0.09906) (layer F.SilkS) (width 0.06604))
-    (fp_line (start -0.09906 -0.09906) (end 0.09906 -0.09906) (layer F.SilkS) (width 0.06604))
-    (fp_line (start -0.09906 0.09906) (end -0.09906 -0.09906) (layer F.SilkS) (width 0.06604))
-    (fp_line (start 0.44958 0.6985) (end 0.79756 0.6985) (layer F.SilkS) (width 0.06604))
-    (fp_line (start 0.79756 0.6985) (end 0.79756 0.44958) (layer F.SilkS) (width 0.06604))
-    (fp_line (start 0.44958 0.44958) (end 0.79756 0.44958) (layer F.SilkS) (width 0.06604))
-    (fp_line (start 0.44958 0.6985) (end 0.44958 0.44958) (layer F.SilkS) (width 0.06604))
-    (fp_line (start 0.79756 0.6985) (end 0.89916 0.6985) (layer F.SilkS) (width 0.06604))
-    (fp_line (start 0.89916 0.6985) (end 0.89916 -0.49784) (layer F.SilkS) (width 0.06604))
-    (fp_line (start 0.79756 -0.49784) (end 0.89916 -0.49784) (layer F.SilkS) (width 0.06604))
-    (fp_line (start 0.79756 0.6985) (end 0.79756 -0.49784) (layer F.SilkS) (width 0.06604))
-    (fp_line (start 0.79756 -0.54864) (end 0.89916 -0.54864) (layer F.SilkS) (width 0.06604))
-    (fp_line (start 0.89916 -0.54864) (end 0.89916 -0.6985) (layer F.SilkS) (width 0.06604))
-    (fp_line (start 0.79756 -0.6985) (end 0.89916 -0.6985) (layer F.SilkS) (width 0.06604))
-    (fp_line (start 0.79756 -0.54864) (end 0.79756 -0.6985) (layer F.SilkS) (width 0.06604))
-    (fp_line (start -0.89916 0.6985) (end -0.79756 0.6985) (layer F.SilkS) (width 0.06604))
-    (fp_line (start -0.79756 0.6985) (end -0.79756 -0.49784) (layer F.SilkS) (width 0.06604))
-    (fp_line (start -0.89916 -0.49784) (end -0.79756 -0.49784) (layer F.SilkS) (width 0.06604))
-    (fp_line (start -0.89916 0.6985) (end -0.89916 -0.49784) (layer F.SilkS) (width 0.06604))
-    (fp_line (start -0.89916 -0.54864) (end -0.79756 -0.54864) (layer F.SilkS) (width 0.06604))
-    (fp_line (start -0.79756 -0.54864) (end -0.79756 -0.6985) (layer F.SilkS) (width 0.06604))
-    (fp_line (start -0.89916 -0.6985) (end -0.79756 -0.6985) (layer F.SilkS) (width 0.06604))
-    (fp_line (start -0.89916 -0.54864) (end -0.89916 -0.6985) (layer F.SilkS) (width 0.06604))
-    (fp_line (start 0.44958 0.6985) (end 0.59944 0.6985) (layer F.SilkS) (width 0.06604))
-    (fp_line (start 0.59944 0.6985) (end 0.59944 0.44958) (layer F.SilkS) (width 0.06604))
-    (fp_line (start 0.44958 0.44958) (end 0.59944 0.44958) (layer F.SilkS) (width 0.06604))
-    (fp_line (start 0.44958 0.6985) (end 0.44958 0.44958) (layer F.SilkS) (width 0.06604))
-    (fp_line (start 1.5494 0.7493) (end -1.5494 0.7493) (layer F.SilkS) (width 0.1016))
-    (fp_line (start -1.5494 0.7493) (end -1.5494 -0.7493) (layer F.SilkS) (width 0.1016))
-    (fp_line (start -1.5494 -0.7493) (end 1.5494 -0.7493) (layer F.SilkS) (width 0.1016))
-    (fp_line (start 1.5494 -0.7493) (end 1.5494 0.7493) (layer F.SilkS) (width 0.1016))
-    (fp_arc (start 0 0) (end 0.54864 0.49784) (angle 95.4) (layer F.SilkS) (width 0.1016))
-    (fp_arc (start 0 0) (end -0.54864 0.49784) (angle 84.5) (layer F.SilkS) (width 0.1016))
-    (fp_arc (start 0 0) (end -0.54864 -0.49784) (angle 95.4) (layer F.SilkS) (width 0.1016))
-    (fp_arc (start 0 0) (end 0.54864 -0.49784) (angle 84.5) (layer F.SilkS) (width 0.1016))
-    (pad 1 smd rect (at -1.41986 0) (size 1.59766 1.80086)
-      (layers F.Cu F.Paste F.Mask)
-    )
-    (pad 2 smd rect (at 1.41986 0) (size 1.59766 1.80086)
-      (layers F.Cu F.Paste F.Mask)
-    )
-  )
-  (module LED-1206 (layer F.Cu)
-    (at 163.957 135.89)
-    (descr "LED 1206 smd package")
-    (tags "LED1206 SMD")
