File: CESP.sch (KiCad schematic (older format))
At the start: 5 parts

Commit message: ADDED/REMOVED SHIT
Parts:
- removed U?: TL074, symbol TL074
- added U?: LM324, symbol LM324
Other:
- moved on the sheet: U?B
Changed lines of the file:
@@
-EESchema Schematic File Version 2  date 1/24/2014 12:04:40 AM
+EESchema Schematic File Version 2
 LIBS:power
 LIBS:device
@@
 Sheet 1 1
 Title ""
-Date "24 jan 2014"
+Date "16 feb 2014"
 Rev ""
 Comp ""
@@
 L TL074 U?
 U 2 1 52E1F3DA
-P 7200 3500
-F 0 "U?" H 7250 3700 60  0000 C CNN
-F 1 "TL074" H 7350 3300 50  0000 C CNN
-F 2 "" H 7200 3500 60  0000 C CNN
-F 3 "" H 7200 3500 60  0000 C CNN
-	2    7200 3500
-	1    0    0    -1
-$EndComp
-$Comp
-L TL074 U?
-U 1 1 52E1F3E5
-P 8600 3500
-F 0 "U?" H 8650 3700 60  0000 C CNN
-F 1 "TL074" H 8750 3300 50  0000 C CNN
-F 2 "" H 8600 3500 60  0000 C CNN
-F 3 "" H 8600 3500 60  0000 C CNN
-	1    8600 3500
+P 8600 4650
+F 0 "U?" H 8650 4850 60  0000 C CNN
+F 1 "TL074" H 8750 4450 50  0000 C CNN
+F 2 "" H 8600 4650 60  0000 C CNN
+F 3 "" H 8600 4650 60  0000 C CNN
+	2    8600 4650
 	1    0    0    -1
 $EndComp
@@
 Text Notes 4450 4650 0    80   ~ 0
 NOTE: THIS IS JUST A TEST BOARD\nREMOVE ALL COMPONENTS AND CREATE YOUR OWN\nINCLUDE SCHEMATIC HOOKUPS/NETLIST
+$Comp
+L LM324 U?
+U 1 1 5300FBFB
+P 3400 4650
+F 0 "U?" H 3450 4850 60  0000 C CNN
+F 1 "LM324" H 3550 4450 50  0000 C CNN
+F 2 "" H 3400 4650 60  0000 C CNN
+F 3 "" H 3400 4650 60  0000 C CNN
+	1    3400 4650
+	1    0    0    -1
+$EndComp
 $EndSCHEMATC
